File: TestLightStrip/fairy_lights_controller.kicad_sch (KiCad schematic)
At the start: 9 parts

Commit message: Updated schematics
Parts:
- Q3, Q4: renamed from Q?; value BC547 -> 2N3904; symbol Transistor_BJT:BC547 -> Transistor_BJT:2N3904
- R3, R4, R5, R6, R7, R8: renamed from R?; footprint (none) -> Resistor_THT:R_Axial_DIN0204_L3.6mm_D1.6mm_P5.08mm_Horizontal
- U2: renamed from U?; value L293 -> L293D
Connections:
- net GND: now also Q3.1 (E), Q4.1 (E); no longer Q3.3 (E), Q4.3 (E)
- net at R6.2, U2.10 (3A): now also Q4.3 (C); no longer Q4.1 (C)
- net at R5.2, U2.2 (1A): now also Q3.3 (C); no longer Q3.1 (C)
Changed lines of the file:
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@@
-(kicad_sch (version 20210126) (generator eeschema)
+(kicad_sch (version 20210406) (generator eeschema)
   (paper "A4")
   (junction (at 96.52 66.04) (diameter 1.016) (color 0 0 0 0))
@@
     (stroke (width 0) (type solid) (color 0 0 0 0))
   )
+  (wire (pts (xy 182.88 82.55) (xy 193.04 82.55))
+    (stroke (width 0) (type solid) (color 0 0 0 0))
+  )
+  (wire (pts (xy 182.88 87.63) (xy 193.04 87.63))
+    (stroke (width 0) (type solid) (color 0 0 0 0))
+  )
+  (wire (pts (xy 182.88 97.79) (xy 193.04 97.79))
+    (stroke (width 0) (type solid) (color 0 0 0 0))
+  )
+  (wire (pts (xy 182.88 102.87) (xy 193.04 102.87))
+    (stroke (width 0) (type solid) (color 0 0 0 0))
+  )
   (hierarchical_label "Select_1" (shape input) (at 83.82 66.04 180)
     (effects (font (size 1.27 1.27)) (justify right))
@@
     (effects (font (size 1.27 1.27)) (justify left))
   )
-  (hierarchical_label "L1_A" (shape bidirectional) (at 182.88 82.55 0)
+  (hierarchical_label "L1_A" (shape bidirectional) (at 193.04 82.55 0)
     (effects (font (size 1.27 1.27)) (justify left))
   )
-  (hierarchical_label "L1_B" (shape bidirectional) (at 182.88 87.63 0)
+  (hierarchical_label "L1_B" (shape bidirectional) (at 193.04 87.63 0)
     (effects (font (size 1.27 1.27)) (justify left))
   )
-  (hierarchical_label "L2_A" (shape bidirectional) (at 182.88 97.79 0)
+  (hierarchical_label "L2_A" (shape bidirectional) (at 193.04 97.79 0)
     (effects (font (size 1.27 1.27)) (justify left))
   )
-  (hierarchical_label "L2_B" (shape bidirectional) (at 182.88 102.87 0)
+  (hierarchical_label "L2_B" (shape bidirectional) (at 193.04 102.87 0)
     (effects (font (size 1.27 1.27)) (justify left))
   )
   (symbol (lib_id "power:+5V") (at 111.76 52.07 0)
     (in_bom yes) (on_board yes)
-    (property "Reference" "#PWR?" (id 0) (at 111.76 55.88 0)
+    (property "Reference" "#PWR07" (id 0) (at 111.76 55.88 0)
       (effects (font (size 1.27 1.27)) hide)
     )
@@
   (symbol (lib_id "power:+5V") (at 111.76 99.06 0)
     (in_bom yes) (on_board yes)
-    (property "Reference" "#PWR?" (id 0) (at 111.76 102.87 0)
+    (property "Reference" "#PWR09" (id 0) (at 111.76 102.87 0)
       (effects (font (size 1.27 1.27)) hide)
     )
@@
   (symbol (lib_id "power:+5V") (at 167.64 72.39 0)
     (in_bom yes) (on_board yes)
-    (property "Reference" "#PWR?" (id 0) (at 167.64 76.2 0)
+    (property "Reference" "#PWR011" (id 0) (at 167.64 76.2 0)
       (effects (font (size 1.27 1.27)) hide)
     )
@@
   (symbol (lib_id "power:GND") (at 111.76 76.2 0)
     (in_bom yes) (on_board yes)
-    (property "Reference" "#PWR?" (id 0) (at 111.76 82.55 0)
+    (property "Reference" "#PWR08" (id 0) (at 111.76 82.55 0)
       (effects (font (size 1.27 1.27)) hide)
     )
@@
   (symbol (lib_id "power:GND") (at 111.76 123.19 0)
     (in_bom yes) (on_board yes)
-    (property "Reference" "#PWR?" (id 0) (at 111.76 129.54 0)
+    (property "Reference" "#PWR010" (id 0) (at 111.76 129.54 0)
       (effects (font (size 1.27 1.27)) hide)
     )
@@
   (symbol (lib_id "power:GND") (at 170.18 123.19 0)
     (in_bom yes) (on_board yes)
-    (property "Reference" "#PWR?" (id 0) (at 170.18 129.54 0)
+    (property "Reference" "#PWR012" (id 0) (at 170.18 129.54 0)
       (effects (font (size 1.27 1.27)) hide)
     )
@@
   (symbol (lib_id "Device:R_Small") (at 101.6 66.04 90)
     (in_bom yes) (on_board yes)
-    (property "Reference" "R?" (id 0) (at 100.9649 63.5 0)
+    (property "Reference" "R3" (id 0) (at 100.9649 63.5 0)
       (effects (font (size 1.27 1.27)) (justify left))
     )
@@
       (effects (font (size 1.27 1.27)) (justify left))
     )
-    (property "Footprint" "" (id 2) (at 101.6 66.04 0)
+    (property "Footprint" "Resistor_THT:R_Axial_DIN0204_L3.6mm_D1.6mm_P5.08mm_Horizontal" (id 2) (at 101.6 66.04 0)
       (effects (font (size 1.27 1.27)) hide)
     )
@@
   (symbol (lib_id "Device:R_Small") (at 101.6 113.03 90)
     (in_bom yes) (on_board yes)
-    (property "Reference" "R?" (id 0) (at 100.9649 110.49 0)
+    (property "Reference" "R4" (id 0) (at 100.9649 110.49 0)
       (effects (font (size 1.27 1.27)) (justify left))
     )
@@
       (effects (font (size 1.27 1.27)) (justify left))
     )
-    (property "Footprint" "" (id 2) (at 101.6 113.03 0)
+    (property "Footprint" "Resistor_THT:R_Axial_DIN0204_L3.6mm_D1.6mm_P5.08mm_Horizontal" (id 2) (at 101.6 113.03 0)
       (effects (font (size 1.27 1.27)) hide)
     )
@@
   (symbol (lib_id "Device:R_Small") (at 111.76 55.88 0)
     (in_bom yes) (on_board yes)
-    (property "Reference" "R?" (id 0) (at 114.3 55.2449 0)
+    (property "Reference" "R5" (id 0) (at 114.3 55.2449 0)
       (effects (font (size 1.27 1.27)) (justify left))
     )
@@
       (effects (font (size 1.27 1.27)) (justify left))
     )
-    (property "Footprint" "" (id 2) (at 111.76 55.88 0)
+    (property "Footprint" "Resistor_THT:R_Axial_DIN0204_L3.6mm_D1.6mm_P5.08mm_Horizontal" (id 2) (at 111.76 55.88 0)
       (effects (font (size 1.27 1.27)) hide)
     )
@@
   (symbol (lib_id "Device:R_Small") (at 111.76 102.87 0)
     (in_bom yes) (on_board yes)
-    (property "Reference" "R?" (id 0) (at 114.3 102.2349 0)
+    (property "Reference" "R6" (id 0) (at 114.3 102.2349 0)
       (effects (font (size 1.27 1.27)) (justify left))
     )
@@
       (effects (font (size 1.27 1.27)) (justify left))
     )
-    (property "Footprint" "" (id 2) (at 111.76 102.87 0)
+    (property "Footprint" "Resistor_THT:R_Axial_DIN0204_L3.6mm_D1.6mm_P5.08mm_Horizontal" (id 2) (at 111.76 102.87 0)
       (effects (font (size 1.27 1.27)) hide)
     )
@@
   (symbol (lib_id "Device:R_Small") (at 152.4 92.71 90) (mirror x)
     (in_bom yes) (on_board yes)
-    (property "Reference" "R?" (id 0) (at 151.13 90.17 90))
+    (property "Reference" "R7" (id 0) (at 151.13 90.17 90))
     (property "Value" "1k" (id 1) (at 151.13 95.25 90))
-    (property "Footprint" "" (id 2) (at 152.4 92.71 0)
+    (property "Footprint" "Resistor_THT:R_Axial_DIN0204_L3.6mm_D1.6mm_P5.08mm_Horizontal" (id 2) (at 152.4 92.71 0)
       (effects (font (size 1.27 1.27)) hide)
     )
@@
   (symbol (lib_id "Device:R_Small") (at 152.4 107.95 90) (mirror x)
     (in_bom yes) (on_board yes)
-    (property "Reference" "R?" (id 0) (at 151.13 105.41 90))
+    (property "Reference" "R8" (id 0) (at 151.13 105.41 90))
     (property "Value" "1k" (id 1) (at 151.13 110.49 90))
-    (property "Footprint" "" (id 2) (at 152.4 107.95 0)
+    (property "Footprint" "Resistor_THT:R_Axial_DIN0204_L3.6mm_D1.6mm_P5.08mm_Horizontal" (id 2) (at 152.4 107.95 0)
       (effects (font (size 1.27 1.27)) hide)
     )
@@
     (pin "2")
   )
-  (symbol (lib_id "Transistor_BJT:BC547") (at 109.22 66.04 0)
-    (in_bom yes) (on_board yes)
-    (property "Reference" "Q?" (id 0) (at 114.3 65.4049 0)
-      (effects (font (size 1.27 1.27)) (justify left))
-    )
-    (property "Value" "BC547" (id 1) (at 114.3 67.9449 0)
+  (symbol (lib_id "Transistor_BJT:2N3904") (at 109.22 66.04 0)
+    (in_bom yes) (on_board yes)
+    (property "Reference" "Q3" (id 0) (at 114.3 65.4049 0)
+      (effects (font (size 1.27 1.27)) (justify left))
+    )
+    (property "Value" "2N3904" (id 1) (at 114.3 67.9449 0)
       (effects (font (size 1.27 1.27)) (justify left))
     )
@@
       (effects (font (size 1.27 1.27) italic) (justify left) hide)
     )
-    (property "Datasheet" "https://www.onsemi.com/pub/Collateral/BC550-D.pdf" (id 3) (at 109.22 66.04 0)
+    (property "Datasheet" "https://www.onsemi.com/pub/Collateral/2N3903-D.PDF" (id 3) (at 109.22 66.04 0)
       (effects (font (size 1.27 1.27)) (justify left) hide)
     )
@@
     (pin "3")
   )
-  (symbol (lib_id "Transistor_BJT:BC547") (at 109.22 113.03 0)
-    (in_bom yes) (on_board yes)
-    (property "Reference" "Q?" (id 0) (at 114.3 112.3949 0)
-      (effects (font (size 1.27 1.27)) (justify left))
-    )
-    (property "Value" "BC547" (id 1) (at 114.3 114.9349 0)
+  (symbol (lib_id "Transistor_BJT:2N3904") (at 109.22 113.03 0)
+    (in_bom yes) (on_board yes)
+    (property "Reference" "Q4" (id 0) (at 114.3 112.3949 0)
+      (effects (font (size 1.27 1.27)) (justify left))
+    )
+    (property "Value" "2N3904" (id 1) (at 114.3 114.9349 0)
       (effects (font (size 1.27 1.27)) (justify left))
     )
@@
       (effects (font (size 1.27 1.27) italic) (justify left) hide)
     )
-    (property "Datasheet" "https://www.onsemi.com/pub/Collateral/BC550-D.pdf" (id 3) (at 109.22 113.03 0)
+    (property "Datasheet" "https://www.onsemi.com/pub/Collateral/2N3903-D.PDF" (id 3) (at 109.22 113.03 0)
       (effects (font (size 1.27 1.27)) (justify left) hide)
     )
@@
   (symbol (lib_id "Driver_Motor:L293") (at 170.18 97.79 0)
     (in_bom yes) (on_board yes)
-    (property "Reference" "U?" (id 0) (at 179.07 71.12 0))
-    (property "Value" "L293" (id 1) (at 177.8 73.66 0))
+    (property "Reference" "U2" (id 0) (at 179.07 71.12 0))
+    (property "Value" "L293D" (id 1) (at 177.8 73.66 0))
     (property "Footprint" "Package_DIP:DIP-16_W7.62mm" (id 2) (at 176.53 116.84 0)
       (effects (font (size 1.27 1.27)) (justify left) hide)
